File: eagle/Mechaduino01_AL3.brd (EAGLE design)
At the start: 41.9 x 41.9 mm, 68 parts, among them IC1 SAMD21G18A-AUT, IC3 LD117AS18TR, Q1 2.5A/30V, Q2 NFET, Q3 BSS138, Q4 BSS138, U3 74AHC1G125, Y1 32,768Khz

Commit message: added readme in /eagle and cleanup
Parts:
- moved C14 3.05 mm to (26.2, 15.0)
- moved C15 3.05 mm to (30.5, 15.0)
- moved R15 2.74 mm to (30.0, 16.4), turned to 270 degrees
- moved R14 2.71 mm to (26.5, 16.4), turned to 270 degrees
- moved C17 1.40 mm to (21.5, 16.4)
- moved C16 1.15 mm to (20.4, 16.4)
- moved C19 0.25 mm to (17.3, 18.7)
- moved U3 0.25 mm to (16.1, 16.3)
- flipped U$4 to the top
Routing:
- net ARDUINO_D13_SCK: track 38.6 -> 63.6 mm, vias 2 -> 3
- net RESET: track 63.7 -> 88.2 mm
- net GND: track 49.7 -> 30.3 mm, vias 52 -> 62
- net ARDUINO_D9----VREF1: track 19.7 -> 25.6 mm
- net ARDUINO_A2----HEADER_SS: track 17.0 -> 22.8 mm, vias 1 -> 2
- net HEADER_SCK: track 10.0 -> 14.1 mm, vias 1 -> 2
- net V+: track 63.8 -> 67.8 mm
- net N$6: track 6.57 -> 3.41 mm
- net N$32: track 6.47 -> 3.46 mm
- net ARDUINO_D4----VREF2: track 26.5 -> 29.2 mm
- net N$27: track 3.79 -> 1.36 mm, vias 1 -> 0
- net HEADER_MOSI: track 8.62 -> 10.9 mm, vias 1 -> 2
- net HEADER_MISO: track 8.72 -> 6.48 mm, vias 1 -> 0
- net N$36: track 32.4 -> 31.5 mm
- net ARDUINO_D8----IN1: track 27.5 -> 28.4 mm
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Other:
- outline, holes or cut-outs redrawn
