File: eagle/Mechaduino01_AL3.sch (EAGLE design)
At the start: 68 parts, among them IC1 SAMD21G18A-AUT, IC2 AP2112K-3.3, Q1 2.5A/30V, Q2 NFET, Q3 BSS138, Q4 BSS138, U3 74AHC1G125, Y1 32,768Khz

Commit message: added readme in /eagle and cleanup
Parts:
- removed IC2: AP2112K-3.3, SparkFun-PowerIC:AP2202-ADJ
- removed SW2: (no value), MF_Switches:TACT_4.2MM
- added IC3: LD117AS18TR, v-reg:LD117AS18TR
- added S1: (no value), _miniRoboter:SMD_SWITCH
- R12, R13: value .25 Ohm -> .15 Ohm
Connections:
- net 3.3V: now also IC3.OUT; no longer IC2.OUT
- net GND: now also IC3.ADJ, S1.P$2; no longer IC2.GND, SW2.P$3, SW2.P$4
- net RESET: now also S1.P$1; no longer SW2.P$1, SW2.P$2
- net VIN: now also IC3.IN; no longer IC2.EN, IC2.IN
Other:
- moved on the sheet: C10, C18
